Commit message: position of the lidar

File: bot_desc/description_gps/gazebo_control.xacro (robot description, xacro)
@@ -19,5 +19,11 @@
         </plugin>
     </gazebo>
-     <gazebo reference="chassis">
+     <gazebo reference="base_link">
+       <material>Gazebo/White</material>
+    </gazebo>
+    <gazebo reference="left_leg_link">
+       <material>Gazebo/White</material>
+    </gazebo>
+    <gazebo reference="right_leg_link">
        <material>Gazebo/White</material>
     </gazebo>

File: bot_desc/description_gps/lidar.xacro (robot description, xacro)
@@ -4,5 +4,5 @@
         <parent link="base_link"/>
         <child link="laser_frame"/>
-        <origin xyz="1.1 0 0.35" rpy="0 0 0"/>
+        <origin xyz="1.25 0 0.35" rpy="0 0.33 0"/>
     </joint>
     <link name="laser_frame">
@@ -39,6 +39,6 @@
                     <horizontal>
                         <samples>360</samples>
-                        <min_angle>-3.14</min_angle>
-                        <max_angle>3.14</max_angle>
+                        <min_angle>-1.17</min_angle>
+                        <max_angle>1.17</max_angle>
                     </horizontal>
                 </scan>
