Commit message: many modification

File: bot_desc/description_gps/robot.urdf.xacro (robot description, xacro)
@@ -1,4 +1,5 @@
 <?xml version="1.0"?>
 <robot xmlns:xacro="http://www.ros.org/wiki/xacro"  name="robot">
+    <!-- <xacro:include filename="robot_core_control.xacro" /> -->
     <xacro:include filename="robot_core.xacro" />
     <xacro:include filename="lidar.xacro" />
@@ -6,4 +7,5 @@
     <xacro:include filename="imu.xacro" />
     <xacro:include filename="gps.xacro" />
-     <xacro:include filename="gazebo_control.xacro" />
+    <!-- <xacro:include filename="ros2_control.xacro" /> -->
+    <xacro:include filename="gazebo_control.xacro" />
 </robot>

File: bot_desc/description_gps_n/ros2_control.xacro (robot description, xacro)
@@ -21,4 +21,20 @@
             <state_interface name="position" />
         </joint>
+        <joint name="wheel_back_right_joint">
+            <command_interface name="velocity">
+                <param name="min">-10</param>
+                <param name="max">10</param>
+            </command_interface>
+            <state_interface name="position" />
+            <state_interface name="velocity" />
+        </joint>
+        <joint name="wheel_back_left_joint">
+            <command_interface name="velocity">
+                <param name="min">-10</param>
+                <param name="max">10</param>
+            </command_interface>
+            <state_interface name="velocity" />
+            <state_interface name="position" />
+        </joint>
         <joint name="left_wheel_leg_joint">
             <command_interface name="position"/>
@@ -27,4 +43,14 @@
         </joint>
         <joint name="right_wheel_leg_joint">
+            <command_interface name="position"/>
+            <state_interface name="position" />
+            <state_interface name="velocity" />
+        </joint>
+        <joint name="left_wheel_back_leg_joint">
+            <command_interface name="position"/>
+            <state_interface name="position" />
+            <state_interface name="velocity" />
+        </joint>
+        <joint name="right_wheel_back_leg_joint">
             <command_interface name="position"/>
             <state_interface name="position" />
