Commit message: Second commit

File: description/robot.urdf.xacro (robot description, xacro)
@@ -5,3 +5,4 @@
     <!--<xacro:include filename="camera.xacro" />-->
     <xacro:include filename="lidar.xacro" />
+    <xacro:include filename="ros2_control.xacro" />
 </robot>

File: description/robot_core.xacro (robot description, xacro)
@@ -61,6 +61,7 @@
 </link>
 <!-- Leg front right-->
-<joint name="leg_front_right_joint" type="fixed">
+<joint name="leg_front_right_joint" type="revolute">
     <origin xyz="0.6 -0.45 -0.5" rpy="0 0 0"/>
+    <limit lower="-0.78" upper="0.78" effort="10" velocity="0.5"/>
     <parent link="base_link"/>
     <child link="leg_front_right_link"/>
@@ -115,5 +116,6 @@
 </link>
 <!-- Leg front left-->
-<joint name="leg_front_left_joint" type="fixed">
+<joint name="leg_front_left_joint" type="revolute">
+    <limit lower="-0.78" upper="0.78" effort="10" velocity="0.5"/>
     <origin xyz="0.6 0.45 -0.5" rpy="0 0 0"/>
     <parent link="base_link"/>

File: description/robot_gazebo.xacro (robot description, xacro)
@@ -5,4 +5,7 @@
     <!-- Gazebo is unable to use the same <material> tags that are already in the URDF (that RViz uses). -->
     <!-- Instead, we need to add gazebo tags for our links that refer to Gazebo materials -->
+    <gazebo reference ="base_footprint">
+            <material>Gazebo/Red</material>
+    </gazebo>
     <gazebo reference="base_link">
         <material>Gazebo/Red</material>
@@ -35,5 +38,5 @@
     <!-- This plugin will publish the joint_states for the selected joints
             (which robot_state_publisher can then use to broadcast the approprate tf). -->
-    <gazebo>
+    <!-- <gazebo>
         <plugin name="gazebo_ros_joint_state_publisher"
             filename="libgazebo_ros_joint_state_publisher.so">
@@ -48,5 +51,5 @@
             <joint_name>wheel_front_right_joint</joint_name>
         </plugin>
-    </gazebo>
+    </gazebo>   -->
     <!-- This plugin will read a JointTrajectory message from the /set_joint_trajectory topic
             and move the machine accordingly. It's a bit clunky but it works. -->
@@ -55,5 +58,5 @@
     <!-- Here's an example message to publish to test it:
             ros2 topic pub -1 /set_joint_trajectory trajectory_msgs/msg/JointTrajectory  '{header: {frame_id: world}, joint_names: [slider_joint, arm_joint], points: [  {positions: {0.8,0.6}} ]}' -->
-     <gazebo>
+     <!-- <gazebo>
         <plugin name="gazebo_ros_joint_pose_trajectory"
             filename="libgazebo_ros_joint_pose_trajectory.so">
@@ -61,4 +64,5 @@
         </plugin>
     </gazebo>
+ -->
         <gazebo>
         <plugin name="diff_drive"
@@ -79,5 +83,5 @@
         </plugin>
     </gazebo>
-    <gazebo>
+    <!-- <gazebo>
     <plugin name="gazebo_ros_control" filename="libgazebo_ros_control.so">
       <robotNamespace>/my_robot</robotNamespace>
@@ -86,6 +90,6 @@
       <alwaysOn>false</alwaysOn>
     </plugin>
-  </gazebo>
-    <gazebo>
+  </gazebo> -->
+   <!--   <gazebo>
      <plugin name="p3d_base_controller" filename="libgazebo_ros_p3d.so">
         <alwaysOn>true</alwaysOn>
@@ -98,4 +102,4 @@
         <rpyOffsets>0 0 0</rpyOffsets>
     </plugin>
-  </gazebo>
+  </gazebo>-->
 </robot>

File: description/ros2_control.xacro (robot description, xacro)
@@ -1,3 +1,45 @@
 <?xml version="1.0"?>
 <robot xmlns:xacro="http://www.ros.org/wiki/xacro">
+    <ros2_control name="GazeboSystem" type="system">
+        <hardware>
+            <plugin>gazebo_ros2_control/GazeboSystem</plugin>
+        </hardware>
+        <joint name="leg_front_left_joint">
+            <command_interface name="position">
+                <param name="min">-10</param>
+                <param name="max">10</param>
+            </command_interface>
+            <state_interface name="position" />
+            <state_interface name="velocity" />
+        </joint>
+        <joint name="leg_front_right_joint">
+            <command_interface name="position">
+                <param name="min">-10</param>
+                <param name="max">10</param>
+            </command_interface>
+            <state_interface name="velocity" />
+            <state_interface name="position" />
+        </joint>
+        <joint name="wheel_front_left_joint">
+            <command_interface name="velocity">
+                <param name="min">-10</param>
+                <param name="max">10</param>
+            </command_interface>
+            <state_interface name="position" />
+            <state_interface name="velocity" />
+        </joint>
+        <joint name="wheel_front_right_joint">
+            <command_interface name="velocity">
+                <param name="min">-10</param>
+                <param name="max">10</param>
+            </command_interface>
+            <state_interface name="velocity" />
+            <state_interface name="position" />
+        </joint>
+    </ros2_control>
+    <gazebo>
+        <plugin name="gazebo_ros2_control" filename="libgazebo_ros2_control.so">
+            <parameters>$(find gps_robot)/config/my_controller.yaml</parameters>
+        </plugin>
+    </gazebo>
 </robot>
